File: HW/QuadUart/QuadUart.kicad_pcb (KiCad board)
At the start: 2 copper layers, 80.3 x 48.7 mm, 100 parts, among them J1 USB_C_Receptacle_USB2.0, J2 Conn_02x05_Odd_Even, J3 Conn_02x10_Odd_Even, J4 Conn_01x05, Q1 BC847, Q2 BC847, SW1 SW_DIP_x04, SW2 SW_DIP_x01, SW3 SW_DIP_x01, U1 LN1134-3.3V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

Commit message: Fixed Input/output swap on buffers, increased to V2
Connections:
- U10 pad 11: /RX_3_RES -> /RX_3_UC
- U10 pad 12: /RX_3_UC -> /RX_3_RES
- U11 pad 11: /DTR_4_UC -> /DTR_4_RES
- U11 pad 12: /DTR_4_RES -> /DTR_4_UC
- U9 pad 11: /DTR_1_UC -> /DTR_1_RES
- U9 pad 12: /DTR_1_RES -> /DTR_1_UC
Routing:
- net /RX_3_UC: track 30.1 -> 30.8 mm
Other:
- board text added: "QuadUart V2 (PIC32MX)"
- board text added: "QuadUart V2 TX/RX/GND/VCC/DTR 2 Banks (2x2 UARTs) /w Power supply 1.8-5.5V"
- board text removed: "QuadUart (PIC32MX)"
- board text removed: "QuadUart TX/RX/GND/VCC/DTR 2 Banks (2x2 UARTs) /w Power supply 1.8-5.5V"
